File: ATU.kicad_pcb (KiCad board)
At the start: 4 copper layers, 100 x 100 mm, 127 parts, among them J1 IN, J2 OUT, J4 12-15V, J5 AVR-ISP-6, K1 G5V-1, K10 G5V-1, K11 G5V-1, K12 G5V-1, K2 G5V-1, K3 G5V-1, K4 G5V-1, K5 G5V-1, K6 G5V-1, K7 G5V-1, K8 G5V-1, K9 G5V-1, Q1 MMBT3904, Q10 MMBT3904, Q11 MMBT3904, Q12 MMBT3904, Q2 MMBT3904, Q3 MMBT3904, Q4 MMBT3904, Q5 MMBT3904, Q6 MMBT3904, Q7 MMBT3904, Q8 MMBT3904, Q9 MMBT3904, SW1 TUNE, SW2 RST, T1 2 x 1:10 T, U1 MCP1703A-5002, U2 ATmega328-AU

Commit message: Backup.
Connections:
- C7 pad 2: REV -> FWD
- C9 pad 1: FWD -> REV
- D2 pad 1: REV -> FWD
- D3 pad 1: FWD -> REV
- R1 pad 2: REV -> FWD
- R4 pad 2: FWD -> REV
- U2 pad 19: FWD -> REV
- U2 pad 22: REV -> FWD
Routing:
- net REV: track 94.1 -> 73.6 mm
- net FWD: track 73.6 -> 94.1 mm
Changed lines of the file:
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@@
       (net 88 "Net-(U2-Pad23)"))
     (pad 22 smd rect (at 4.25 -1.2 45) (size 1.6 0.55) (layers F.Cu F.Paste F.Mask)
-      (net 8 REV))
+      (net 10 FWD))
     (pad 21 smd rect (at 4.25 -0.4 45) (size 1.6 0.55) (layers F.Cu F.Paste F.Mask)
       (net 1 GND))
@@
       (net 23 "Net-(C25-Pad1)"))
     (pad 19 smd rect (at 4.25 1.2 45) (size 1.6 0.55) (layers F.Cu F.Paste F.Mask)
-      (net 10 FWD))
+      (net 8 REV))
     (pad 18 smd rect (at 4.25 2 45) (size 1.6 0.55) (layers F.Cu F.Paste F.Mask)
       (net 22 +5VA))
@@
     (fp_line (start -1.6 0.8) (end -1.6 -0.8) (layer F.Fab) (width 0.1))
     (pad 2 smd roundrect (at 1.4875 0 270) (size 1.425 1.75) (layers F.Cu F.Paste F.Mask) (roundrect_rratio 0.175439)
-      (net 10 FWD))
+      (net 8 REV))
     (pad 1 smd roundrect (at -1.4875 0 270) (size 1.425 1.75) (layers F.Cu F.Paste F.Mask) (roundrect_rratio 0.175439)
       (net 9 "Net-(C8-Pad1)"))
@@
     (fp_line (start -1.6 0.8) (end -1.6 -0.8) (layer F.Fab) (width 0.1))
     (pad 2 smd roundrect (at 1.4875 0 270) (size 1.425 1.75) (layers F.Cu F.Paste F.Mask) (roundrect_rratio 0.175439)
-      (net 8 REV))
+      (net 10 FWD))
     (pad 1 smd roundrect (at -1.4875 0 270) (size 1.425 1.75) (layers F.Cu F.Paste F.Mask) (roundrect_rratio 0.175439)
       (net 7 "Net-(C6-Pad2)"))
@@
     )
     (pad 1 smd rect (at 1 0 180) (size 0.9 0.8) (layers F.Cu F.Paste F.Mask)
-      (net 10 FWD))
+      (net 8 REV))
     (pad "" smd rect (at -1 0.95 180) (size 0.9 0.8) (layers F.Cu F.Paste F.Mask))
     (pad 2 smd rect (at -1 -0.95 180) (size 0.9 0.8) (layers F.Cu F.Paste F.Mask)
@@
     )
     (pad 1 smd rect (at 1 0) (size 0.9 0.8) (layers F.Cu F.Paste F.Mask)
-      (net 8 REV))
+      (net 10 FWD))
     (pad "" smd rect (at -1 0.95) (size 0.9 0.8) (layers F.Cu F.Paste F.Mask))
     (pad 2 smd rect (at -1 -0.95) (size 0.9 0.8) (layers F.Cu F.Paste F.Mask)
@@
       (net 1 GND))
     (pad 1 smd roundrect (at -1.4875 0) (size 1.425 1.75) (layers F.Cu F.Paste F.Mask) (roundrect_rratio 0.175439)
-      (net 10 FWD))
+      (net 8 REV))
     (model ${KISYS3DMOD}/Capacitor_SMD.3dshapes/C_1206_3216Metric.wrl
       (at (xyz 0 0 0))
@@
     (fp_line (start -1.6 0.8) (end -1.6 -0.8) (layer F.Fab) (width 0.1))
     (pad 2 smd roundrect (at 1.4875 0 270) (size 1.425 1.75) (layers F.Cu F.Paste F.Mask) (roundrect_rratio 0.175439)
-      (net 8 REV))
+      (net 10 FWD))
     (pad 1 smd roundrect (at -1.4875 0 270) (size 1.425 1.75) (layers F.Cu F.Paste F.Mask) (roundrect_rratio 0.175439)
       (net 1 GND))
@@
   (segment (start 50.1 98.82) (end 46.29 98.82) (width 0.5) (layer F.Cu) (net 6))
   (segment (start 69.785 48.02) (end 69.785 53.935) (width 0.25) (layer F.Cu) (net 7))
-  (segment (start 92.075 111.585) (end 92.01 111.52) (width 0.25) (layer F.Cu) (net 8))
-  (segment (start 92.075 121.822944) (end 92.075 111.585) (width 0.25) (layer F.Cu) (net 8))
-  (segment (start 90.991676 122.906268) (end 92.075 121.822944) (width 0.25) (layer F.Cu) (net 8))
-  (segment (start 92.01 111.52) (end 93.28 111.52) (width 0.25) (layer F.Cu) (net 8))
-  (segment (start 93.28 111.52) (end 93.28 111.52) (width 0.25) (layer F.Cu) (net 8))
-  (via (at 93.28 111.52) (size 0.8) (drill 0.4) (layers F.Cu B.Cu) (net 8))
-  (segment (start 72.96 59.45) (end 72.96 59.45) (width 0.25) (layer B.Cu) (net 8))
-  (segment (start 93.679999 111.120001) (end 93.28 111.52) (width 0.25) (layer B.Cu) (net 8))
-  (segment (start 93.679999 59.849999) (end 93.679999 111.120001) (width 0.25) (layer B.Cu) (net 8))
-  (segment (start 93.28 59.45) (end 93.679999 59.849999) (width 0.25) (layer B.Cu) (net 8))
-  (segment (start 69.785 59.45) (end 93.28 59.45) (width 0.25) (layer B.Cu) (net 8))
-  (via (at 69.785 59.45) (size 0.8) (drill 0.4) (layers F.Cu B.Cu) (net 8))
-  (segment (start 67.245 56.91) (end 69.785 56.91) (width 0.25) (layer F.Cu) (net 8))
-  (segment (start 69.785 56.91) (end 69.785 59.45) (width 0.25) (layer F.Cu) (net 8))
+  (segment (start 92.075 111.585) (end 92.01 111.52) (width 0.25) (layer F.Cu) (net 10))
+  (segment (start 92.075 121.822944) (end 92.075 111.585) (width 0.25) (layer F.Cu) (net 10))
+  (segment (start 90.991676 122.906268) (end 92.075 121.822944) (width 0.25) (layer F.Cu) (net 10))
+  (segment (start 92.01 111.52) (end 93.28 111.52) (width 0.25) (layer F.Cu) (net 10))
+  (segment (start 93.28 111.52) (end 93.28 111.52) (width 0.25) (layer F.Cu) (net 10))
+  (via (at 93.28 111.52) (size 0.8) (drill 0.4) (layers F.Cu B.Cu) (net 10))
+  (segment (start 72.96 59.45) (end 72.96 59.45) (width 0.25) (layer B.Cu) (net 10))
+  (segment (start 93.679999 111.120001) (end 93.28 111.52) (width 0.25) (layer B.Cu) (net 10))
+  (segment (start 93.679999 59.849999) (end 93.679999 111.120001) (width 0.25) (layer B.Cu) (net 10))
+  (segment (start 93.28 59.45) (end 93.679999 59.849999) (width 0.25) (layer B.Cu) (net 10))
+  (segment (start 69.785 59.45) (end 93.28 59.45) (width 0.25) (layer B.Cu) (net 10))
+  (via (at 69.785 59.45) (size 0.8) (drill 0.4) (layers F.Cu B.Cu) (net 10))
+  (segment (start 67.245 56.91) (end 69.785 56.91) (width 0.25) (layer F.Cu) (net 10))
+  (segment (start 69.785 56.91) (end 69.785 59.45) (width 0.25) (layer F.Cu) (net 10))
   (segment (start 97.72 52.025) (end 97.725 52.03) (width 0.25) (layer F.Cu) (net 9))
   (segment (start 95.185 52.025) (end 97.72 52.025) (width 0.25) (layer F.Cu) (net 9))
   (segment (start 97.725 52.03) (end 97.725 49.29) (width 0.25) (layer F.Cu) (net 9))
-  (segment (start 96.455 120.837056) (end 96.455 111.52) (width 0.25) (layer F.Cu) (net 10))
-  (segment (start 92.688732 124.603324) (end 96.455 120.837056) (width 0.25) (layer F.Cu) (net 10))
-  (segment (start 96.455 111.52) (end 94.55 111.52) (width 0.25) (layer F.Cu) (net 10))
-  (segment (start 94.55 111.52) (end 94.55 111.52) (width 0.25) (layer F.Cu) (net 10))
-  (via (at 94.55 111.52) (size 0.8) (drill 0.4) (layers F.Cu B.Cu) (net 10))
-  (segment (start 95.185 59.45) (end 95.185 59.45) (width 0.25) (layer B.Cu) (net 10))
-  (via (at 95.185 59.45) (size 0.8) (drill 0.4) (layers F.Cu B.Cu) (net 10))
-  (segment (start 94.150001 60.72) (end 95.185 59.45) (width 0.25) (layer B.Cu) (net 10))
-  (segment (start 94.150001 111.120001) (end 94.150001 60.72) (width 0.25) (layer B.Cu) (net 10))
-  (segment (start 94.55 111.52) (end 94.150001 111.120001) (width 0.25) (layer B.Cu) (net 10))
-  (segment (start 95.185 55) (end 95.185 59.45) (width 0.25) (layer F.Cu) (net 10))
+  (segment (start 96.455 120.837056) (end 96.455 111.52) (width 0.25) (layer F.Cu) (net 8))
+  (segment (start 92.688732 124.603324) (end 96.455 120.837056) (width 0.25) (layer F.Cu) (net 8))
+  (segment (start 96.455 111.52) (end 94.55 111.52) (width 0.25) (layer F.Cu) (net 8))
+  (segment (start 94.55 111.52) (end 94.55 111.52) (width 0.25) (layer F.Cu) (net 8))
+  (via (at 94.55 111.52) (size 0.8) (drill 0.4) (layers F.Cu B.Cu) (net 8))
+  (segment (start 95.185 59.45) (end 95.185 59.45) (width 0.25) (layer B.Cu) (net 8))
+  (via (at 95.185 59.45) (size 0.8) (drill 0.4) (layers F.Cu B.Cu) (net 8))
+  (segment (start 94.150001 60.72) (end 95.185 59.45) (width 0.25) (layer B.Cu) (net 8))
+  (segment (start 94.150001 111.120001) (end 94.150001 60.72) (width 0.25) (layer B.Cu) (net 8))
+  (segment (start 94.55 111.52) (end 94.150001 111.120001) (width 0.25) (layer B.Cu) (net 8))
+  (segment (start 95.185 55) (end 95.185 59.45) (width 0.25) (layer F.Cu) (net 8))
   (segment (start 87.24401 122.340583) (end 86.295 121.391573) (width 0.25) (layer F.Cu) (net 11))
   (segment (start 83.444073 121.391573) (end 80.7975 118.745) (width 0.25) (layer F.Cu) (net 11))
